File: kicad/micro-esp32-s3.kicad_pcb (KiCad board)
At the start: 2 copper layers, 48 x 35.1 mm, 69 parts, among them IC1 IRM-H638T/TR2, J1 TYPE-C-31-M-12, J3 DM3D-SF, Q1 NTA4151PT1G, Q2 NTA4151PT1G, Q3 NTA4151PT1G, U1 NCP167BMX330TBG, U2 ESP32-S3-WROOM-1, U3 MAX98357AETE+T, U4 TP4057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

Commit message: Fix diode position
Parts:
- R10: value 100K -> 1K
- moved D6 2.54 mm to (95.2, 98.6), turned to -90 degrees
- moved Q2 0.25 mm to (97.0, 98.9), turned to -90 degrees
Connections:
- C2 pad 1: Net-(Q2-S) -> Net-(D6-K)
- D6 pad 1: BAT+ -> Net-(D6-K)
- Q2 pad 2: Net-(Q2-S) -> Net-(D6-K)
- U1 pad 3: Net-(Q2-S) -> Net-(D6-K)
- U1 pad 4: Net-(Q2-S) -> Net-(D6-K)
Routing:
- net Net-(D6-K): track 0.00 -> 4.52 mm
- net Net-(Q2-S): track 3.90 -> 0.00 mm
- net +5V: track 79.0 -> 79.9 mm, vias 7 -> 9
- net BAT+: track 34.8 -> 33.8 mm

Commit message: WIP - version 3
Parts:
- added C19: 1uF, Capacitor_SMD:C_0402_1005Metric, F.Cu at (105.9, 105.2)
- added Q4: TPNTA4153NT1G, Package_TO_SOT_SMD:SOT-523, F.Cu at (109.6, 100.1)
- added R25: 12K, Resistor_SMD:R_0402_1005Metric, F.Cu at (109.7, 102.0)
- R10: value 1K -> 12K
- R20: value 12K -> 10K
- U6: value ~ -> USBLC6-2P6; footprint Connector_PinHeader_2.54mm:PinHeader_1x08_P2.54mm_Vertical -> Package_TO_SOT_SMD:SOT-666
- moved D3 39.1 mm to (135.1, 123.7)
- moved R5 39.1 mm to (132.5, 122.7)
- moved R6 39.1 mm to (135.1, 122.7)
- moved D2 39.1 mm to (132.5, 123.8)
- moved D4 38.9 mm to (137.4, 123.7)
- moved R8 38.9 mm to (137.4, 122.7)
- moved R21 36.6 mm to (133.1, 95.4)
- moved Q3 35.9 mm to (133.1, 99.0), turned to -90 degrees
- moved R20 34.7 mm to (133.1, 93.1)
- moved R22 34.6 mm to (133.1, 94.2)
- moved R19 34.5 mm to (133.1, 92.0)
- moved R14 34.1 mm to (133.1, 96.8), turned to 0 degrees
- moved R12 31.4 mm to (94.9, 96.5)
- moved C15 30.6 mm to (99.1, 96.6), turned to 180 degrees
- moved Y1 30.6 mm to (102.2, 95.8), turned to 180 degrees
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Connections:
- net Net-(D1-K) renamed AMP_VDD
- net Net-(D6-K) renamed BUS_PWR
- QWIIC1 pad 3: IO44 -> IO5
- QWIIC1 pad 4: IO42 -> IO4
- QWIIC2 pad 3: IO2 -> IO6
- QWIIC2 pad 4: IO43 -> IO7
- R10 pad 1: MASS_STORAGE_EN -> VDD33
- R10 pad 2: GND -> Net-(Q4-D)
- U2 pad 10: TFT_MOSI -> SD_CARD_DAT1
- U2 pad 11: TFT_PWR -> SD_CARD_DAT0
- U2 pad 12: TFT_SCLK -> SD_CARD_PWR
- U2 pad 15: ~{SD_MODE} -> unconnected-(U2-GPIO3/TOUCH3/ADC1_CH2-Pad15)
- U2 pad 16: IO46 -> unconnected-(U2-GPIO46-Pad16)
- U2 pad 17: SPK_DIN -> SD_CARD_CMD
- U2 pad 18: SPK_BCLK -> SD_CARD_DAT3
- U2 pad 19: SPK_LRCLK -> SD_CARD_DAT2
- U2 pad 20: BUILT_IN_LED -> ~{SD_MODE}
- U2 pad 21: IR_PWR -> SPK_DIN
- U2 pad 22: IR_IN -> SPK_BCLK
- U2 pad 23: SD_CARD_PWR -> SPK_LRCLK
- U2 pad 24: SD_CARD_DAT1 -> IR_IN
- U2 pad 25: SD_CARD_DAT0 -> IR_PWR
- U2 pad 26: IO45 -> unconnected-(U2-GPIO45-Pad26)
- U2 pad 28: SD_CARD_CLK -> unconnected-(U2-SPIIO6/GPIO35/FSPID/SUBSPID-Pad28)
- U2 pad 29: SD_CARD_CMD -> unconnected-(U2-SPIIO7/GPIO36/FSPICLK/SUBSPICLK-Pad29)
- U2 pad 30: SD_CARD_DAT3 -> unconnected-(U2-SPIDQS/GPIO37/FSPIQ/SUBSPIQ-Pad30)
- U2 pad 31: SD_CARD_DAT2 -> BUILT_IN_LED
- U2 pad 32: MASS_STORAGE_EN -> TFT_RST
- U2 pad 33: unconnected-(U2-MTDO/GPIO40/CLK_OUT2-Pad33) -> TFT_MOSI
- U2 pad 34: unconnected-(U2-MTDI/GPIO41/CLK_OUT1-Pad34) -> TFT_SCLK
- U2 pad 35: IO42 -> TFT_CS
- U2 pad 36: IO44 -> TFT_DC
- U2 pad 37: IO43 -> TFT_PWR
- U2 pad 38: IO2 -> BAT_MONITOR
- U2 pad 39: unconnected-(U2-GPIO1/TOUCH1/ADC1_CH0-Pad39) -> USB_PWR_DETECT
- U2 pad 4: USB_PWR_DETECT -> IO4
- U2 pad 5: BAT_MONITOR -> IO5
- U2 pad 6: TFT_BLK -> IO6
- U2 pad 7: TFT_CS -> IO7
- U2 pad 8: TFT_DC -> MASS_STORAGE_EN
- U2 pad 9: TFT_RST -> SD_CARD_CLK
- U5 pad 18: MASS_STORAGE_EN -> Net-(Q4-D)
- U6 pad 1: GND -> USB_D+
- U6 pad 2: TFT_VCC -> GND
- U6 pad 3: TFT_SCLK -> USB_D-
- U6 pad 4: TFT_MOSI -> USB_D-
- U6 pad 5: TFT_RST -> +5V
- U6 pad 6: TFT_DC -> USB_D+
Routing:
- net VDD33: track 120.8 -> 24.7 mm, vias 9 -> 2
- net GND: track 65.5 -> 0.00 mm, vias 62 -> 0
- net TFT_VCC: track 57.3 -> 6.52 mm, vias 3 -> 1
- net TFT_RST: track 44.0 -> 11.7 mm, vias 2 -> 1
- net BAT+: track 33.8 -> 65.8 mm, vias 1 -> 6
- net TFT_SCLK: track 43.1 -> 11.7 mm
- net TFT_CS: track 42.7 -> 12.0 mm, vias 2 -> 1
- net TFT_MOSI: track 42.1 -> 11.5 mm, vias 2 -> 1
- net TFT_DC: track 41.9 -> 11.8 mm
- net +5V: track 79.9 -> 106.9 mm, vias 9 -> 6
- net Net-(U5-LED): track 48.8 -> 30.3 mm, vias 4 -> 0
- net USB_D-: track 46.7 -> 65.2 mm, vias 4 -> 2
- net MASS_STORAGE_EN: track 20.4 -> 4.11 mm, vias 4 -> 0
- net USB_D+: track 48.1 -> 64.1 mm, vias 4 -> 2
- net SPK-: track 3.88 -> 19.5 mm
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- removed copper zone on B.Cu, net GND
- removed copper zone on F.Cu, net GND

Commit message: V3 Work in progress
Parts:
- added C20: 100nF, Capacitor_SMD:C_0402_1005Metric, F.Cu at (116.6, 116.1)
- moved D7 2.18 mm to (123.7, 113.3)
- moved D1 2.11 mm to (125.0, 113.3)
- moved C11 1.94 mm to (95.7, 98.4), turned to 180 degrees
- moved R15 1.17 mm to (117.0, 113.0)
- moved R12 1.14 mm to (96.0, 96.5)
- moved D3 0.62 mm to (135.0, 124.4)
- moved R6 0.62 mm to (135.0, 123.3)
- moved D2 0.61 mm to (132.5, 124.4)
- moved D4 0.61 mm to (137.4, 124.4)
- moved R5 0.61 mm to (132.5, 123.3)
- moved R8 0.61 mm to (137.4, 123.3)
- moved U6 0.54 mm to (114.8, 115.8), turned to 90 degrees
- moved D5 0.13 mm to (95.3, 124.5)
- moved R9 0.13 mm to (95.3, 123.4)
- turned R10 to -90 degrees
Connections:
- J1 pad A6: USB_D+ -> USB_D_IN+
- J1 pad A7: USB_D- -> USB_D_IN-
- J1 pad B6: USB_D+ -> USB_D_IN+
- J1 pad B7: USB_D- -> USB_D_IN-
- SPK1 pad 1: SPK+ -> SPK-
- SPK1 pad 2: SPK- -> SPK+
- U6 pad 1: USB_D+ -> USB_D_IN-
- U6 pad 3: USB_D- -> USB_D_IN+
- U6 pad 4: USB_D- -> USB_D+
- U6 pad 6: USB_D+ -> USB_D-
Routing:
- net GND: track 0.00 -> 102.4 mm, vias 0 -> 64
- net USB_D-: track 65.2 -> 38.2 mm
- net USB_D+: track 64.1 -> 38.7 mm
- net USB_D_IN-: track 0.00 -> 6.54 mm
- net +5V: track 106.9 -> 101.1 mm, vias 6 -> 7
- net SPK-: track 19.5 -> 25.0 mm
- net USB_D_IN+: track 0.00 -> 5.24 mm
- net VDD33: track 24.7 -> 29.0 mm, vias 2 -> 10
- net Net-(U5-RBIAS): track 0.00 -> 3.86 mm
- net AMP_VDD: track 5.95 -> 9.15 mm
- net BAT+: track 65.8 -> 68.0 mm
- net Net-(U3-~{SD_MODE}): track 0.00 -> 2.14 mm
- net SPK+: track 21.8 -> 23.4 mm
- net SD_CARD_PWR: track 3.17 -> 4.77 mm
- net SD_CARD_CLK: track 38.8 -> 40.3 mm
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- added copper zone on F.Cu, net GND
- added copper zone on In1.Cu, net GND
- added copper zone on In2.Cu, net VDD33
Other:
- copper layers 2 -> 4

Commit message: Version 3 - Ready for review
Parts:
- removed the QWIIC1 at (107.6, 95.7)
- added C21: 100nF, Capacitor_SMD:C_0402_1005Metric, F.Cu at (109.6, 120.3)
- added G***: LOGO, qwiic:qwiic, B.Cu at (105.2, 121.2)
- added U8: OWMMOD-403010A-S261F, OWMMOD-403010A-S261F:MIC_OWMMOD-403010A-S261F, F.Cu at (109.3, 122.9)
- U2: footprint PCM_Espressif:ESP32-S3-WROOM-1 -> PCM_Espressif:ESP32-S3-WROOM-1U
- moved QWIIC1 29.5 mm to (99.7, 120.3), turned to 180 degrees
- moved R16 29.1 mm to (98.8, 123.7), turned to -90 degrees
- moved C14 29.0 mm to (97.7, 123.7), turned to 90 degrees
- moved C15 27.6 mm to (104.4, 123.7), turned to -90 degrees
- moved Y1 27.4 mm to (101.6, 123.2), turned to 0 degrees
- moved R12 25.9 mm to (105.0, 120.8), turned to 0 degrees
- moved C16 24.9 mm to (102.9, 120.8), turned to 0 degrees
- moved R24 23.7 mm to (99.7, 120.8), turned to 180 degrees
- moved R23 22.5 mm to (96.4, 119.4), turned to 180 degrees
- moved C11 16.4 mm to (96.5, 114.8)
- moved C12 16.3 mm to (105.9, 115.7), turned to 0 degrees
- moved C10 16.3 mm to (106.0, 119.5)
- moved U5 15.1 mm to (101.2, 116.5), turned to 180 degrees
- moved Q4 13.0 mm to (108.7, 113.0), turned to -90 degrees
- moved C19 11.8 mm to (96.8, 112.6)
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- renumbered QWIIC2 to QWIIC1
Connections:
- QWIIC1 pad 3: IO6 -> SDA
- QWIIC1 pad 4: IO7 -> SCL
- U2 pad 10: SD_CARD_DAT1 -> SD_CARD_DAT2
- U2 pad 11: SD_CARD_DAT0 -> SCL
- U2 pad 12: SD_CARD_PWR -> SDA
- U2 pad 15: unconnected-(U2-GPIO3/TOUCH3/ADC1_CH2-Pad15) -> MASS_STORAGE_EN
- U2 pad 17: SD_CARD_CMD -> MIC_LR
- U2 pad 18: SD_CARD_DAT3 -> MIC_CLK
- U2 pad 19: SD_CARD_DAT2 -> MIC_DATA
- U2 pad 4: IO4 -> SD_CARD_DAT1
- U2 pad 5: IO5 -> SD_CARD_DAT0
- U2 pad 6: IO6 -> SD_CARD_CLK
- U2 pad 7: IO7 -> SD_CARD_PWR
- U2 pad 8: MASS_STORAGE_EN -> SD_CARD_CMD
- U2 pad 9: SD_CARD_CLK -> SD_CARD_DAT3
Routing:
- net GND: track 102.4 -> 124.1 mm, vias 64 -> 78
- net SDA: track 0.00 -> 21.6 mm, vias 0 -> 1
- net SCL: track 0.00 -> 21.4 mm, vias 0 -> 1
- net MIC_DATA: track 0.00 -> 18.2 mm, vias 0 -> 2
- net MIC_CLK: track 0.00 -> 17.8 mm, vias 0 -> 2
- net MIC_LR: track 0.00 -> 16.5 mm, vias 0 -> 2
- net USB_D+: track 38.7 -> 25.1 mm
- net USB_D-: track 38.2 -> 26.5 mm
- net Net-(U5-LED): track 30.2 -> 18.5 mm, vias 0 -> 2
- net SPK-: track 25.0 -> 14.0 mm
- net SPK+: track 23.4 -> 12.6 mm
- net SD_CARD_DAT3: track 41.6 -> 32.5 mm, vias 4 -> 2
- net SD_CARD_DAT2: track 41.7 -> 33.2 mm, vias 4 -> 2
- net SD_CARD_CMD: track 38.2 -> 31.0 mm
- net IO7: track 7.18 -> 0.00 mm, vias 1 -> 0
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- added copper zone on B.Cu, net GND
Other:
- board text added: "3V3"
- board text added: "DISPLAY"
- board text added: "ESP32-TV Version 3 atomic14"
- board text added: "SCL"
- board text added: "SDA"
- board text removed: "ESP32-TV Version 2 atomic14"
- board text removed: "QWIIC1"
- board text removed: "QWIIC2"

Commit message: Submitted Version
Parts:
- added R26: 10K, Resistor_SMD:R_0402_1005Metric, F.Cu at (102.1, 95.1)
- added R27: 10K, Resistor_SMD:R_0402_1005Metric, F.Cu at (100.8, 95.1)
- added R28: 10K, Resistor_SMD:R_0402_1005Metric, F.Cu at (99.6, 95.1)
- added R29: 10K, Resistor_SMD:R_0402_1005Metric, F.Cu at (97.0, 95.1)
- added R30: 10K, Resistor_SMD:R_0402_1005Metric, F.Cu at (98.3, 95.1)
- added R31: 10K, Resistor_SMD:R_0402_1005Metric, F.Cu at (95.8, 95.1)
- C1, C20, C21, C8: value 100nF -> 0.1uF
- D2: value LED -> RED
- D3: value LED -> GREEN
- D4: value LED -> BLUE
- D5: value LED -> YELLOW
- moved R15 0.63 mm to (116.5, 113.4)
Connections:
- net Net-(J3-VDD) renamed SD_CARD_VDD
Routing:
- net SD_CARD_VDD: track 14.6 -> 33.1 mm
- net SD_CARD_DAT2: track 33.2 -> 46.4 mm, vias 2 -> 5
- net SD_CARD_DAT3: track 32.5 -> 44.7 mm, vias 2 -> 4
- net SD_CARD_CMD: track 31.0 -> 42.2 mm, vias 2 -> 3
- net SD_CARD_CLK: track 34.3 -> 41.7 mm, vias 2 -> 3
- net SD_CARD_DAT0: track 42.2 -> 48.5 mm
- net SD_CARD_DAT1: track 42.5 -> 47.7 mm
- net ~{SD_MODE}: track 5.77 -> 6.44 mm
- net GND: vias 78 -> 76
Other:
- board text added: "WayWayWay"
