File: kicad/micro-esp32-s3.kicad_sch (KiCad schematic)
At the start: 69 parts, among them IC1 IRM-H638T/TR2, J1 TYPE-C-31-M-12, J3 DM3D-SF, Q1 NTA4151PT1G, Q2 NTA4151PT1G, Q3 NTA4151PT1G, U1 NCP167BMX330TBG, U2 ESP32-S3-WROOM-1, U3 MAX98357AETE+T, U4 TP4057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

Commit message: WIP - version 3
Parts:
- removed U6: ~, Connector_PinHeader_2.54mm:PinHeader_1x08_P2.54mm_Vertical, symbol display:1.69_Rounded
- added C19: 1uF, Capacitor_SMD:C_0402_1005Metric, symbol Device:C_Small
- added Q4: TPNTA4153NT1G, Package_TO_SOT_SMD:SOT-523, symbol Device:Q_NMOS_GSD
- added R25: 12K, Resistor_SMD:R_0402_1005Metric, symbol Device:R_Small
- added U6: USBLC6-2P6, Package_TO_SOT_SMD:SOT-666, symbol Power_Protection:USBLC6-2P6
- IC1: footprint SOP254P700X405-4N -> IRM-H638M3_TR2:SOP254P700X405-4N
- J3: footprint DM3DSF -> DM3D-SF:DM3DSF
- R10: value 1K -> 12K
- R20: value 12K -> 10K
Connections:
- net TFT_BLK is gone; now on net IO6: U2.6 (GPIO6/TOUCH6/ADC1_CH5)
- net +3V3: now also R10.1, R25.1
- net +5V: now also U6.5 (VBUS)
- net BAT_MONITOR: now also U2.38 (GPIO2/TOUCH2/ADC1_CH1); no longer U2.5 (GPIO5/TOUCH5/ADC1_CH4)
- net BUILT_IN_LED: now also U2.31 (GPIO38/FSPIWP/SUBSPIWP); no longer U2.20 (GPIO12/TOUCH12/ADC2_CH1/FSPICLK/FSPIIO6/SUBSPICLK)
- net GND: now also C19.2, Q4.2 (S), U6.2 (GND); no longer R10.2
- net IR_IN: now also U2.24 (GPIO47/SPICLK_P/SUBSPICLK_P_DIFF); no longer U2.22 (GPIO14/TOUCH14/ADC2_CH3/FSPIWP/FSPIDQS/SUBSPIWP)
- net IR_PWR: now also U2.25 (GPIO48/SPICLK_N/SUBSPICLK_N_DIFF); no longer U2.21 (GPIO13/TOUCH13/ADC2_CH2/FSPIQ/FSPIIO7/SUBSPIQ)
- net MASS_STORAGE_EN: now also U2.8 (GPIO15/U0RTS/ADC2_CH4/XTAL_32K_P), Q4.1 (G), R25.2; no longer R10.1, U2.32 (MTCK/GPIO39/CLK_OUT3/SUBSPICS1), U5.18 (~{RESET})
- net SD_CARD_CLK: now also U2.9 (GPIO16/U0CTS/ADC2_CH5/XTAL_32K_N); no longer U2.28 (SPIIO6/GPIO35/FSPID/SUBSPID)
- net SD_CARD_CMD: now also U2.17 (GPIO9/TOUCH9/ADC1_CH8/FSPIHD/SUBSPIHD); no longer U2.29 (SPIIO7/GPIO36/FSPICLK/SUBSPICLK)
- net SD_CARD_DAT0: now also U2.11 (GPIO18/U1RXD/ADC2_CH7/CLK_OUT3); no longer U2.25 (GPIO48/SPICLK_N/SUBSPICLK_N_DIFF)
- net SD_CARD_DAT1: now also U2.10 (GPIO17/U1TXD/ADC2_CH6); no longer U2.24 (GPIO47/SPICLK_P/SUBSPICLK_P_DIFF)
- net SD_CARD_DAT2: now also U2.19 (GPIO11/TOUCH11/ADC2_CH0/FSPID/FSPIIO5/SUBSPID); no longer U2.31 (GPIO38/FSPIWP/SUBSPIWP)
- net SD_CARD_DAT3: now also U2.18 (GPIO10/TOUCH10/ADC1_CH9/FSPICS0/FSPIIO4/SUBSPICS0); no longer U2.30 (SPIDQS/GPIO37/FSPIQ/SUBSPIQ)
- net SD_CARD_PWR: now also U2.12 (GPIO8/TOUCH8/ADC1_CH7/SUBSPICS1); no longer U2.23 (GPIO21)
- net SPK_BCLK: now also U2.22 (GPIO14/TOUCH14/ADC2_CH3/FSPIWP/FSPIDQS/SUBSPIWP); no longer U2.18 (GPIO10/TOUCH10/ADC1_CH9/FSPICS0/FSPIIO4/SUBSPICS0)
- net SPK_DIN: now also U2.21 (GPIO13/TOUCH13/ADC2_CH2/FSPIQ/FSPIIO7/SUBSPIQ); no longer U2.17 (GPIO9/TOUCH9/ADC1_CH8/FSPIHD/SUBSPIHD)
- net SPK_LRCLK: now also U2.23 (GPIO21); no longer U2.19 (GPIO11/TOUCH11/ADC2_CH0/FSPID/FSPIIO5/SUBSPID)
- net TFT_CS: now also U2.35 (MTMS/GPIO42); no longer U2.7 (GPIO7/TOUCH7/ADC1_CH6)
- net TFT_DC: now also U2.36 (U0RXD/GPIO44/CLK_OUT2); no longer U2.8 (GPIO15/U0RTS/ADC2_CH4/XTAL_32K_P)
- net TFT_MOSI: now also U2.33 (MTDO/GPIO40/CLK_OUT2); no longer U2.10 (GPIO17/U1TXD/ADC2_CH6)
- net TFT_PWR: now also U2.37 (U0TXD/GPIO43/CLK_OUT1); no longer U2.11 (GPIO18/U1RXD/ADC2_CH7/CLK_OUT3)
- net TFT_RST: now also U2.32 (MTCK/GPIO39/CLK_OUT3/SUBSPICS1); no longer U2.9 (GPIO16/U0CTS/ADC2_CH5/XTAL_32K_N)
- net TFT_SCLK: now also U2.34 (MTDI/GPIO41/CLK_OUT1); no longer U2.12 (GPIO8/TOUCH8/ADC1_CH7/SUBSPICS1)
- net USB_D+: now also U6.1 (I/O1), U6.6 (I/O1)
- net USB_D-: now also U6.3 (I/O2), U6.4 (I/O2)
- net USB_PWR_DETECT: now also U2.39 (GPIO1/TOUCH1/ADC1_CH0); no longer U2.4 (GPIO4/TOUCH4/ADC1_CH3)
- net ~{SD_MODE}: now also U2.20 (GPIO12/TOUCH12/ADC2_CH1/FSPICLK/FSPIIO6/SUBSPICLK); no longer U2.15 (GPIO3/TOUCH3/ADC1_CH2)
- net BUS_PWR: now reaches C2.1, D6.1 (K), Q2.2 (S), U1.3 (EN), U1.4 (IN)
- net AMP_VDD: now reaches C7.1, C8.1, D1.1 (K), D7.1 (K), U3.7 (VDD), U3.8 (VDD)
- net IO2 renamed IO6
- net IO6: no longer U2.38 (GPIO2/TOUCH2/ADC1_CH1)
- net IO42 renamed IO4
- net IO4: now also U2.4 (GPIO4/TOUCH4/ADC1_CH3); no longer U2.35 (MTMS/GPIO42)
- net IO43 renamed IO7
- net IO7: now also U2.7 (GPIO7/TOUCH7/ADC1_CH6); no longer U2.37 (U0TXD/GPIO43/CLK_OUT1)
- net IO44 renamed IO5
- net IO5: now also U2.5 (GPIO5/TOUCH5/ADC1_CH4); no longer U2.36 (U0RXD/GPIO44/CLK_OUT2)
- new net: C19.1, Q4.3 (D), R10.2, U5.18 (~{RESET})
Other:
- note removed: "Need to find a suitable value for this. There appears to be an undocumented internal pullup resistor on the reset pin."
- moved on the sheet: C10, C11, C12, C13, C14, C15, C16, C17, C4, C9, D4, D5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

Commit message: V3 Work in progress
Parts:
- added C20: 100nF, Capacitor_SMD:C_0402_1005Metric, symbol Device:C_Small
Connections:
- net +5V: now also C20.1
- net GND: now also C20.2
- net SPK+: now also SPK1.2; no longer SPK1.1
- net SPK-: now also SPK1.1; no longer SPK1.2
- net USB_D+: now also U6.4 (I/O2); no longer J1.A6 (DP1), J1.B6 (DP2), U6.1 (I/O1), U6.6 (I/O1)
- net USB_D-: now also U6.6 (I/O1); no longer J1.A7 (DN1), J1.B7 (DN2), U6.3 (I/O2), U6.4 (I/O2)
- new net USB_D_IN+: J1.A6 (DP1), J1.B6 (DP2), U6.3 (I/O2)
- new net USB_D_IN-: J1.A7 (DN1), J1.B7 (DN2), U6.1 (I/O1)

Commit message: Version 3 - Ready for review
Parts:
- removed QWIIC1: SM04B-SRSS-TB_LF__SN_, SM04B-SRSS-TB_LF__SN_:JST_SM04B-SRSS-TB_LF__SN_, symbol SM04B-SRSS-TB_LF__SN_:SM04B-SRSS-TB_LF__SN_
- added C21: 100nF, Capacitor_SMD:C_0402_1005Metric, symbol Device:C_Small
- added U8: OWMMOD-403010A-S261F, OWMMOD-403010A-S261F:MIC_OWMMOD-403010A-S261F, symbol OWMMOD-403010A-S261F:OWMMOD-403010A-S261F
- U2: footprint PCM_Espressif:ESP32-S3-WROOM-1 -> PCM_Espressif:ESP32-S3-WROOM-1U
- renumbered QWIIC2 to QWIIC1
Connections:
- net IO4 is gone; now on net SD_CARD_DAT1: U2.4 (GPIO4/TOUCH4/ADC1_CH3)
- net IO5 is gone; now on net SD_CARD_DAT0: U2.5 (GPIO5/TOUCH5/ADC1_CH4)
- net +3V3: now also C21.1, U8.3 (VDD)
- net GND: now also C21.2, U8.5 (GND), U8.6 (GND), U8.7 (GND), U8.8 (GND)
- net MASS_STORAGE_EN: now also U2.15 (GPIO3/TOUCH3/ADC1_CH2); no longer U2.8 (GPIO15/U0RTS/ADC2_CH4/XTAL_32K_P)
- net SD_CARD_CLK: now also U2.6 (GPIO6/TOUCH6/ADC1_CH5); no longer U2.9 (GPIO16/U0CTS/ADC2_CH5/XTAL_32K_N)
- net SD_CARD_CMD: now also U2.8 (GPIO15/U0RTS/ADC2_CH4/XTAL_32K_P); no longer U2.17 (GPIO9/TOUCH9/ADC1_CH8/FSPIHD/SUBSPIHD)
- net SD_CARD_DAT0: no longer U2.11 (GPIO18/U1RXD/ADC2_CH7/CLK_OUT3)
- net SD_CARD_DAT1: no longer U2.10 (GPIO17/U1TXD/ADC2_CH6)
- net SD_CARD_DAT2: now also U2.10 (GPIO17/U1TXD/ADC2_CH6); no longer U2.19 (GPIO11/TOUCH11/ADC2_CH0/FSPID/FSPIIO5/SUBSPID)
- net SD_CARD_DAT3: now also U2.9 (GPIO16/U0CTS/ADC2_CH5/XTAL_32K_N); no longer U2.18 (GPIO10/TOUCH10/ADC1_CH9/FSPICS0/FSPIIO4/SUBSPICS0)
- net SD_CARD_PWR: now also U2.7 (GPIO7/TOUCH7/ADC1_CH6); no longer U2.12 (GPIO8/TOUCH8/ADC1_CH7/SUBSPICS1)
- net IO6 renamed SDA
- net SDA: now also U2.12 (GPIO8/TOUCH8/ADC1_CH7/SUBSPICS1); no longer U2.6 (GPIO6/TOUCH6/ADC1_CH5)
- net IO7 renamed SCL
- net SCL: now also U2.11 (GPIO18/U1RXD/ADC2_CH7/CLK_OUT3); no longer U2.7 (GPIO7/TOUCH7/ADC1_CH6)
- new net MIC_CLK: U2.18 (GPIO10/TOUCH10/ADC1_CH9/FSPICS0/FSPIIO4/SUBSPICS0), U8.1 (CLK)
- new net MIC_DATA: U2.19 (GPIO11/TOUCH11/ADC2_CH0/FSPID/FSPIIO5/SUBSPID), U8.2 (DATA)
- new net MIC_LR: U2.17 (GPIO9/TOUCH9/ADC1_CH8/FSPIHD/SUBSPIHD), U8.4 (L/R)
Other:
- moved on the sheet: BAT1, C18, C20, C4, IC1, J1, J3, Q1, Q3, QWIIC1, R11, R13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

Commit message: Submitted Version
Parts:
- added R26, R27, R28, R29, R30, R31: 10K, Resistor_SMD:R_0402_1005Metric, symbol Device:R_Small
- C1, C20, C21, C8: value 100nF -> 0.1uF
- D2: value LED -> RED
- D3: value LED -> GREEN
- D4: value LED -> BLUE
- D5: value LED -> YELLOW
Connections:
- net SD_CARD_CLK: now also R30.1
- net SD_CARD_CMD: now also R28.1
- net SD_CARD_DAT0: now also R31.1
- net SD_CARD_DAT1: now also R29.1
- net SD_CARD_DAT2: now also R26.1
- net SD_CARD_DAT3: now also R27.1
- net SD_CARD_VDD: now reaches J3.4 (VDD), Q1.3 (D)
- net SD_CARD_VDD: now also R26.2, R27.2, R28.2, R29.2, R30.2, R31.2
